File: KiCad/_autosave-Helios.kicad_pcb (KiCad board)
At the start: 2 copper layers, 99.5 x 88 mm, 72 parts, among them CON1 AVR-JTAG-10, J1 Conn_01x04, J10 Conn_01x10, J11 Conn_01x16, J2 Conn_01x04, J3 Conn_01x04, J4 Conn_01x04, J5 Conn_01x04, J6 Conn_01x04, J7 Conn_01x11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

Commit message: start board routing
Parts:
- moved F2 2.80 mm to (169.2, 72.9)
- moved RV2 2.73 mm to (169.2, 68.6)
- moved RV1 0.45 mm to (168.5, 55.8)
- moved F1 0.28 mm to (168.6, 60.9)
Routing:
- added copper zone on B.Cu, net GND
Changed lines of the file:
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@@
   (general
     (links 260)
-    (no_connects 260)
-    (area 88.982893 45.215765 189.582895 133.315767)
+    (no_connects 255)
+    (area -65.040001 -28.360001 189.875001 206.860001)
     (thickness 1.6)
     (drawings 180)
@@
   )
   (module Resistors_SMD:R_1210_HandSoldering (layer F.Cu)
-    (at 168.3 56.2)
+    (at 168.5 55.8)
     (descr "Resistor SMD 1210, hand soldering")
     (tags "resistor 1210")
@@
   )
   (module Resistors_SMD:R_1210_HandSoldering (layer F.Cu)
-    (at 168.8 65.9)
+    (at 169.2 68.6)
     (descr "Resistor SMD 1210, hand soldering")
     (tags "resistor 1210")
@@
   )
   (module Resistors_SMD:R_1812 (layer F.Cu)
-    (at 168.4 60.7)
+    (at 168.6 60.9)
     (descr "Resistor SMD 1812, flow soldering, Panasonic (see ERJ12)")
     (tags "resistor 1812")
@@
   )
   (module Resistors_SMD:R_1812 (layer F.Cu)
-    (at 169.1 70.1)
+    (at 169.2 72.9)
     (descr "Resistor SMD 1812, flow soldering, Panasonic (see ERJ12)")
     (tags "resistor 1812")
@@
   (gr_arc (start 187.032894 103.465763) (end 186.519864 102.056224) (angle -5.841933) (layer Edge.Cuts) (width 0.1))
   (gr_arc (start 187.032894 103.465763) (end 186.379059 102.115763) (angle -64.158069) (layer Edge.Cuts) (width 0.1))
+  (zone (net 2) (net_name GND) (layer B.Cu) (hatch edge 0.508)
+    (connect_pads (clearance 0.508))
+    (min_thickness 0.254)
+    (fill yes (arc_segments 16) (thermal_gap 0.508) (thermal_bridge_width 0.508))
+    (polygon
+      (pts
+        (xy 85.3 136.5) (xy 193.1 136.5) (xy 193.9 36.8) (xy 84.2 36.3) (xy 80.6 133.3)
+      )
+    )
+  )
 )
