File: KiCad/Helios.kicad_pcb (KiCad board)
At the start: 2 copper layers, 99.5 x 91.2 mm, 74 parts, among them CON1 AVR-JTAG-10, J1 Conn_01x04, J10 Conn_01x10, J11 GS3, J12 GS3, J13 GS3, J2 Conn_01x04, J3 Conn_01x04, J4 Conn_01x04, J5 Conn_01x04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

Commit message: make sure everything is up to date before transfer to CodeCommit
Parts:
- removed J10: Conn_01x10, Pin_Headers:Pin_Header_Straight_1x10_Pitch2.54mm
- removed J11, J12, J13: GS3, Connectors:GS3
- removed J9: Conn_01x09, Pin_Headers:Pin_Header_Straight_1x09_Pitch2.54mm
- added F5: Polyfuse_Small, Resistor_SMD:R_1812_4532Metric, F.Cu at (98.0, 58.6)
- added Q1: Q_NMOS_GDS, Package_TO_SOT_SMD:SOT-223-3_TabPin2, F.Cu at (178.8, 96.1)
- added R13: 10k, Resistor_SMD:R_1206_3216Metric, F.Cu at (151.9, 80.0)
- added R14: 125, Resistor_SMD:R_1206_3216Metric, F.Cu at (97.0, 65.3)
- added R15: 10k, Resistor_SMD:R_1206_3216Metric, F.Cu at (183.2, 61.1)
- added R16: 10k, Resistor_SMD:R_1206_3216Metric, F.Cu at (183.2, 66.0)
- added SW1: SW_DPDT_x2, CH20M:DPDT, F.Cu at (165.1, 60.6)
- added SW2: SW_DPDT_x2, CH20M:DPDT, F.Cu at (174.9, 60.6)
- C13, C16, C19, C22, C25: value 100nF -> .1uF
- D4: footprint Diodes_SMD:D_1206 -> Diode_SMD:D_1206_3216Metric
- J2: footprint CH20M:CH20Mt -> CH20M:CH20Mr
- J5: footprint CH20M:CH20Mr -> CH20M:CH20Mt
- J7: value Conn_01x11 -> Conn_02x10_Counter_Clockwise; footprint Pin_Headers:Pin_Header_Straight_1x11_Pitch2.54mm -> Package_DIP:DIP-20_W7.62mm_Socket
- moved J2 80.7 mm to (152.4, 126.6), turned to 180 degrees
- moved J5 80.6 mm to (152.0, 52.0), turned to 0 degrees
- moved D4 35.6 mm to (102.7, 65.4)
- moved J4 30.1 mm to (121.9, 52.0)
- moved J3 30.0 mm to (182.4, 126.6)
- moved J7 15.9 mm to (95.3, 74.9), turned to 0 degrees
- moved C1 7.15 mm to (113.0, 93.5)
- moved J8 7.10 mm to (184.9, 77.2)
- moved U1 5.49 mm to (114.7, 78.7)
- moved F1 5.40 mm to (170.3, 73.7)
- moved D3 5.40 mm to (163.7, 75.2)
- moved RV1 5.40 mm to (178.1, 73.7)
- moved F2 5.40 mm to (170.5, 79.0)
- moved RV2 5.40 mm to (178.1, 79.0)
- moved CON1 2.92 mm to (157.6, 97.4)
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Connections:
- D4 pad 1: +3V3 -> Net-(D4-Pad1)
- D4 pad 2: Net-(D4-Pad2) -> GND
- D5 pad 1: Net-(D4-Pad2) -> Net-(D5-Pad1)
- F4 pad 1: Net-(D4-Pad2) -> Net-(D5-Pad1)
- J2 pad 1: Net-(D2-Pad2) -> RTDb1
- J2 pad 2: GNDPWR -> RTDb2
- J2 pad 3: GND -> RTDb3
- J2 pad 4: /Pyro -> RTDb4
- J3 pad 1: RTDb1 -> RTD-1
- J3 pad 2: RTDb2 -> RTD-2
- J3 pad 3: RTDb3 -> RTD-3
- J3 pad 4: RTDb4 -> RTD-4
- J4 pad 1: /RS485A -> Net-(D2-Pad2)
- J4 pad 2: /RS485B -> GNDPWR
- J4 pad 4: /Wind -> /Pyro
- J5 pad 1: RTD-1 -> /RS485A
- J5 pad 2: RTD-2 -> /RS485B
- J5 pad 3: RTD-3 -> GND
- J5 pad 4: RTD-4 -> /Wind
- J7 pad 1: Net-(J7-Pad1) -> GND
- J7 pad 10: Net-(J7-Pad10) -> +24V
- J7 pad 11: Net-(J7-Pad11) -> +24V
- J7 pad 2: Net-(J7-Pad2) -> /GPIOB/MOSI
- J7 pad 3: Net-(J7-Pad3) -> /GPIOB/SCK
- J7 pad 4: Net-(J7-Pad4) -> /GPIOB/~CS
- J7 pad 5: Net-(J7-Pad5) -> /GPIOB/D/~C
- J7 pad 7: Net-(J7-Pad7) -> /GPIOB/485TX
- J7 pad 8: Net-(J7-Pad8) -> /GPIOB/485RX
- J7 pad 9: Net-(J7-Pad9) -> +3V3
- R5 pad 1: Net-(D4-Pad2) -> Net-(D5-Pad1)
- U2 pad 23: Net-(J7-Pad1) -> Net-(U2-Pad23)
- U2 pad 29: Net-(J7-Pad2) -> Net-(U2-Pad29)
- U2 pad 30: Net-(J7-Pad3) -> Net-(U2-Pad30)
- U2 pad 31: Net-(J7-Pad4) -> Net-(U2-Pad31)
- U2 pad 32: Net-(J7-Pad5) -> Net-(U2-Pad32)
- U2 pad 51: /GPIOB/~RST -> Net-(U2-Pad51)
- U2 pad 60: Net-(D4-Pad2) -> Net-(D5-Pad1)
- U2 pad 61: Net-(U2-Pad61) -> Net-(D4-Pad1)
- U2 pad 67: Net-(J7-Pad6) -> Net-(U2-Pad67)
- U2 pad 68: Net-(J7-Pad7) -> Net-(U2-Pad68)
- U2 pad 69: Net-(J7-Pad8) -> Net-(U2-Pad69)
- U2 pad 70: Net-(J7-Pad9) -> Net-(U2-Pad70)
- U2 pad 71: Net-(J7-Pad10) -> Net-(U2-Pad71)
- U2 pad 77: Net-(J7-Pad11) -> Net-(U2-Pad77)
Routing:
- net WindDir: track 0.00 -> 81.6 mm
- net /GPIOB/~RST: track 76.7 -> 0.00 mm, vias 1 -> 0
- net Net-(D4-Pad1): track 0.00 -> 74.4 mm
- net Net-(J7-Pad6): track 58.7 -> 0.00 mm, vias 1 -> 0
- net Net-(J7-Pad10): track 56.6 -> 0.00 mm, vias 1 -> 0
- net Net-(J7-Pad9): track 55.5 -> 0.00 mm, vias 1 -> 0
- net Net-(J7-Pad8): track 54.8 -> 0.00 mm, vias 1 -> 0
- net Net-(J7-Pad7): track 54.4 -> 0.00 mm, vias 1 -> 0
- net Net-(J7-Pad5): track 53.8 -> 0.00 mm
- net Net-(J7-Pad11): track 52.0 -> 0.00 mm, vias 1 -> 0
- net +24V: track 49.4 -> 101.2 mm
- net Net-(D4-Pad2): track 46.0 -> 0.00 mm, vias 2 -> 0
- net Net-(J7-Pad3): track 45.2 -> 0.00 mm
- net /Snow: track 46.3 -> 91.5 mm
- net Net-(J7-Pad4): track 42.5 -> 0.00 mm
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- removed copper zone on B.Cu, net GND
- removed copper zone on F.Cu, net GND
Other:
- outline, holes or cut-outs redrawn
- board text added: "Helios Test board V1.0"
- board text added: "RTD"
- board text added: "WX"
- board text removed: "Helios Test board V0.6"

Commit message: submittal of circuit board for assembly
Parts:
- C10: value .1u -> .1 uF; footprint Capacitors_SMD:C_1206_HandSoldering -> Capacitor_SMD:C_1206_3216Metric
- C11, C12, C14, C15, C17, C18, C20, C21, C23, C24: footprint Capacitors_SMD:C_1206_HandSoldering -> Capacitor_SMD:C_1206_3216Metric
- C13, C16, C19, C22, C25, C3, C5, C7, C9: value .1uF -> .1 uF; footprint Capacitors_SMD:C_1206_HandSoldering -> Capacitor_SMD:C_1206_3216Metric
- C2, C4, C6, C8: value 1uF -> 1 uF; footprint Capacitors_SMD:C_1206_HandSoldering -> Capacitor_SMD:C_1206_3216Metric
- D1, D2, D5, D6, D7, D8, D9: footprint Diodes_SMD:D_1206 -> Diode_SMD:D_1206_3216Metric
- D3: footprint TO_SOT_Packages_SMD:SOT-23_Handsoldering -> Package_TO_SOT_SMD:SOT-23
- F1, F2, F3, F4: footprint Resistors_SMD:R_1812 -> Resistor_SMD:R_1812_4532Metric
- J8: footprint Pin_Headers:Pin_Header_Straight_1x06_Pitch2.54mm -> Connector_PinSocket_2.54mm:PinSocket_1x06_P2.54mm_Vertical
- R1, R10, R11, R12, R4, R6, R7, R8, R9: footprint Resistors_SMD:R_1206_HandSoldering -> Resistor_SMD:R_1206_3216Metric
- R14: value 125 -> 120
- R2, R3: value 10 -> TBU; footprint Resistors_SMD:R_1812_HandSoldering -> CH20M:TBU
- R5: value 125 -> 120; footprint Resistors_SMD:R_1206_HandSoldering -> Resistor_SMD:R_1206_3216Metric
- RV1, RV2: footprint Resistors_SMD:R_1210_HandSoldering -> Resistor_SMD:R_1210_3225Metric
- moved R4 14.6 mm to (173.0, 85.6), turned to 0 degrees
- moved R6 13.1 mm to (178.5, 85.6)
- moved R5 10.6 mm to (134.8, 61.1)
- moved C17 9.68 mm to (146.2, 106.3)
- moved C9 9.30 mm to (123.2, 84.8)
- moved C23 7.64 mm to (180.2, 105.2)
- moved R13 7.27 mm to (158.7, 82.6)
- moved C24 6.82 mm to (174.1, 105.1), turned to 0 degrees
- moved D2 5.64 mm to (111.8, 57.2)
- moved D1 5.47 mm to (116.8, 57.3)
- moved C18 5.32 mm to (139.3, 106.3), turned to 0 degrees
- moved C8 5.19 mm to (123.2, 92.3), turned to 90 degrees
- moved C4 4.60 mm to (147.6, 101.0), turned to 0 degrees
- moved R1 4.40 mm to (113.3, 63.0)
- moved C21 2.48 mm to (157.2, 104.9)
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Connections:
- J7 pad 15: Net-(J7-Pad15) -> /GPIOF/~reset
- J7 pad 6: Net-(J7-Pad6) -> /GPIOF/~reset
- Q1 pad 2: GND -> /Snow
- Q1 pad 3: /Snow -> GND
- U2 pad 11: Net-(U2-Pad11) -> /GPIOF/~reset
Routing:
- net GND: track 599.1 -> 0.00 mm, vias 2 -> 0
- net +3V3: track 374.8 -> 0.00 mm, vias 7 -> 0
- net RTD_MISO: track 122.3 -> 0.00 mm, vias 3 -> 0
- net RTD_SCK: track 119.0 -> 0.00 mm, vias 3 -> 0
- net RTD_MOSI: track 118.0 -> 0.00 mm, vias 3 -> 0
- net RTD-1: track 104.7 -> 0.00 mm
- net +24V: track 101.2 -> 0.00 mm
- net /Snow: track 91.5 -> 0.00 mm, vias 1 -> 0
- net WindDir: track 81.6 -> 0.00 mm
- net /GPIOB/SCK: track 78.1 -> 0.00 mm, vias 1 -> 0
- net RTD-5: track 75.8 -> 0.00 mm
- net Net-(D4-Pad1): track 74.4 -> 0.00 mm
- net RTD-2: track 71.7 -> 0.00 mm
- net RTDb5: track 69.4 -> 0.00 mm, vias 2 -> 0
- net RTDb1: track 64.1 -> 0.00 mm, vias 1 -> 0
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